File: Capacitor MMC/Capacitor MMC.kicad_pcb (KiCad board)
At the start: 2 copper layers, 215.9 x 63.5 mm, 10 parts, among them J1 Screw_Terminal_01x01, J2 Screw_Terminal_01x01

Commit message: add mounting holes to capacitor board
Parts:
- added H1: MountingHole, MountingHole:MountingHole_5mm_Pad, F.Cu at (39.4, 71.1)
- added H2: MountingHole, MountingHole:MountingHole_5mm_Pad, F.Cu at (166.6, 46.3)
- added H3: MountingHole, MountingHole:MountingHole_5mm_Pad, F.Cu at (177.1, 35.8)
- added H4: MountingHole, MountingHole:MountingHole_5mm_Pad, F.Cu at (177.1, 46.3)
Changed lines of the file:
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@@
-(kicad_pcb (version 20171130) (host pcbnew "(5.1.4)-1")
+(kicad_pcb (version 20171130) (host pcbnew 5.0.2+dfsg1-1)
   (general
     (thickness 1.6)
@@
     (tracks 29)
     (zones 0)
-    (modules 10)
+    (modules 14)
     (nets 6)
   )
@@
   )
   (setup
-    (last_trace_width 12.7)
+    (last_trace_width 0.25)
     (user_trace_width 2.54)
     (user_trace_width 12.7)
@@
     (zone_45_only no)
     (trace_min 0.2)
+    (segment_width 0.2)
+    (edge_width 0.05)
     (via_size 0.8)
     (via_drill 0.4)
@@
     (uvia_min_size 0.2)
     (uvia_min_drill 0.1)
-    (edge_width 0.05)
-    (segment_width 0.2)
     (pcb_text_width 0.3)
     (pcb_text_size 1.5 1.5)
@@
     )
   )
+  (module MountingHole:MountingHole_5mm_Pad (layer F.Cu)
+    (at 39.37 71.12)
+    (descr "Mounting Hole 5mm")
+    (tags "mounting hole 5mm")
+    (attr virtual)
+    (fp_text reference H1 (at 0 -6) (layer F.SilkS)
+      (effects (font (size 1 1) (thickness 0.15)))
+    )
+    (fp_text value MountingHole (at 0 6) (layer F.Fab)
+      (effects (font (size 1 1) (thickness 0.15)))
+    )
+    (fp_text user %R (at 0.3 0) (layer F.Fab)
+      (effects (font (size 1 1) (thickness 0.15)))
+    )
+    (fp_circle (center 0 0) (end 5 0) (layer Cmts.User) (width 0.15))
+    (fp_circle (center 0 0) (end 5.25 0) (layer F.CrtYd) (width 0.05))
+    (pad 1 thru_hole circle (at 0 0) (size 10 10) (drill 5) (layers *.Cu *.Mask))
+  )
+  (module MountingHole:MountingHole_5mm_Pad (layer F.Cu)
+    (at 166.565001 46.305001)
+    (descr "Mounting Hole 5mm")
+    (tags "mounting hole 5mm")
+    (attr virtual)
+    (fp_text reference H2 (at 0 -6) (layer F.SilkS)
+      (effects (font (size 1 1) (thickness 0.15)))
+    )
+    (fp_text value MountingHole (at 0 6) (layer F.Fab)
+      (effects (font (size 1 1) (thickness 0.15)))
+    )
+    (fp_circle (center 0 0) (end 5.25 0) (layer F.CrtYd) (width 0.05))
+    (fp_circle (center 0 0) (end 5 0) (layer Cmts.User) (width 0.15))
+    (fp_text user %R (at 0.3 0) (layer F.Fab)
+      (effects (font (size 1 1) (thickness 0.15)))
+    )
+    (pad 1 thru_hole circle (at 0 0) (size 10 10) (drill 5) (layers *.Cu *.Mask))
+  )
+  (module MountingHole:MountingHole_5mm_Pad (layer F.Cu)
+    (at 177.115001 35.755001)
+    (descr "Mounting Hole 5mm")
+    (tags "mounting hole 5mm")
+    (attr virtual)
+    (fp_text reference H3 (at 0 -6) (layer F.SilkS)
+      (effects (font (size 1 1) (thickness 0.15)))
+    )
+    (fp_text value MountingHole (at 0 6) (layer F.Fab)
+      (effects (font (size 1 1) (thickness 0.15)))
+    )
+    (fp_text user %R (at 0.3 0) (layer F.Fab)
+      (effects (font (size 1 1) (thickness 0.15)))
+    )
+    (fp_circle (center 0 0) (end 5 0) (layer Cmts.User) (width 0.15))
+    (fp_circle (center 0 0) (end 5.25 0) (layer F.CrtYd) (width 0.05))
+    (pad 1 thru_hole circle (at 0 0) (size 10 10) (drill 5) (layers *.Cu *.Mask))
+  )
+  (module MountingHole:MountingHole_5mm_Pad (layer F.Cu)
+    (at 177.115001 46.305001)
+    (descr "Mounting Hole 5mm")
+    (tags "mounting hole 5mm")
+    (attr virtual)
+    (fp_text reference H4 (at 0 -6) (layer F.SilkS)
+      (effects (font (size 1 1) (thickness 0.15)))
+    )
+    (fp_text value MountingHole (at 0 6) (layer F.Fab)
+      (effects (font (size 1 1) (thickness 0.15)))
+    )
+    (fp_circle (center 0 0) (end 5.25 0) (layer F.CrtYd) (width 0.05))
+    (fp_circle (center 0 0) (end 5 0) (layer Cmts.User) (width 0.15))
+    (fp_text user %R (at 0.3 0) (layer F.Fab)
+      (effects (font (size 1 1) (thickness 0.15)))
+    )
+    (pad 1 thru_hole circle (at 0 0) (size 10 10) (drill 5) (layers *.Cu *.Mask))
+  )
   (gr_line (start 25.4 127) (end 25.4 63.5) (layer Edge.Cuts) (width 0.05))
